File: PCB/board.sch (EAGLE design)
At the start: 38 parts, among them IC1 W25Q32JVSSIQ, J1 USB-TYPE-C-31-M-12, Q1 S8050, Q2 S8050, U1 AMS1117_SOT223, U2 CH340C, U3 ESP8266EX, X1 SMA, Y1 40Mhz

Commit message: library update
Parts:
- U3: device angrypig7-IC:ESP8266EX -> angrypig7-IC-MCU:ESP8266EX
Changed lines of the file:
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@@
 <part name="SUPPLY3" library="SparkFun-PowerSymbols" deviceset="5V" device=""/>
 <part name="GND3" library="SparkFun-PowerSymbols" deviceset="GND" device=""/>
-<part name="U3" library="angrypig7-IC" deviceset="ESP8266EX" device="">
+<part name="U3" library="angrypig7-IC-MCU" deviceset="ESP8266EX" device="">
 <attribute name="LCSC" value="C77967"/>
 </part>
